File: Extero75.kicad_pcb (KiCad board)
At the start: 2 copper layers, 362 x 142.9 mm, 314 parts, among them J1 USB_C_Receptacle_USB2.0, Q1 AO3400A, SW1 BOOT, SW2 RST, SW3 RotaryEncoder_Switch, U1 STM32F072R8Tx, U2 XC6206P332MR

Commit message: some more routing
Parts:
- C12, C13, C14, C15, C16, C2, C3, C4, C5, C6, C7, C8, C9, D1, D10, D11, D12, D13, D14, D15, D16, D17, D18, D19, D2, D20, D21, D22, D23, D24, D25, D26, D27, D28, D29, D3, D30, D31, D32, D33, D34, D35, D36, D37, D38, D39, D4, D40, D41, D42, D43, D44, D45, D46, D47, D48, D49, D5, D50, D51, D52, D53, D54, D55, D56, D57, D58, D59, D6, D60, D61, D62, D63, D64, D65, D66, D67, D68, D69, D7, D70, D71, D72, D73, D74, D75, D76, D77, D78, D79, D8, D80, D81, D82, D83, D84, D85, D86, D87, D88, D89, D9, D90, D91, D92, D93, D94, D95, Q1, R1, R101, R11, R13, R14, R15, R17, R18, R19, R2, R20, R21, R23, R25, R26, R3, R30, R31, R32, R33, R36, R37, R4, R40, R42, R44, R45, R47, R5, R52, R53, R54, R55, R56, R57, R58, R59, R60, R62, R63, R64, R65, R67, R69, R7, R73, R74, R75, R77, R78, R79, R8, R80, R81, R82, R84, R85, R88, R89, R91, R93, R94, R95, R97, R98, R99, SW1, SW2, U1, U2: moved to B.Cu
- moved R4 568.8 mm to (-724.0, 19.3), turned to -90 degrees
- moved C2 559.7 mm to (-602.0, 127.0), turned to -90 degrees
- moved D4 559.5 mm to (-752.0, 105.8)
- moved C14 543.2 mm to (-559.9, 134.2), turned to 180 degrees
- moved R18 540.6 mm to (-708.9, 28.9), turned to 180 degrees
- moved D8 537.8 mm to (-733.1, 67.5)
- moved R5 534.9 mm to (-727.1, 19.3), turned to -90 degrees
- moved C13 518.8 mm to (-559.9, 133.1), turned to 180 degrees
- moved D1 507.9 mm to (-752.7, 48.4)
- moved D15 504.4 mm to (-699.9, 67.7)
- moved D12 503.7 mm to (-701.4, 15.5)
- moved D19 486.1 mm to (-682.1, 48.7)
- moved D5 483.9 mm to (-752.4, 124.6)
- moved D3 479.3 mm to (-752.4, 86.6)
- moved D20 468.7 mm to (-675.0, 125.0)
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Connections:
- net Net-(C1-Pad1) renamed /BOOT
- net Net-(C2-Pad1) renamed /RST
- C12 pad 1: +3V3 -> +3.3V
- C13 pad 1: +3V3 -> +3.3V
- C14 pad 1: +3V3 -> +3.3V
- C15 pad 1: +3V3 -> +3.3V
- C16 pad 1: +3V3 -> +3.3V
- C8 pad 1: +3V3 -> +3.3V
- C9 pad 1: +3V3 -> +3.3V
- MX-J1 pad 1: unconnected-(MX-J1-Pad1) -> COL9
- MX-U1 pad 1: unconnected-(MX-U1-Pad1) -> COL9
- Num1 pad 3: unconnected-(Num1-Pad3) -> Net-(Num1-Pad3)
- Num7 pad 1: unconnected-(Num7-Pad1) -> COL9
- R21 pad 2: unconnected-(R21-Pad2) -> LED-
- R25 pad 1: unconnected-(R25-Pad1) -> Net-(Num1-Pad3)
- Tab1 pad 4: unconnected-(Tab1-Pad4) -> +5V
- U1 pad 10: unconnected-(U1-Pad10) -> ROW5
- U1 pad 14: COL12 -> unconnected-(U1-Pad14)
- U1 pad 26: D_N -> unconnected-(U1-Pad26)
- U1 pad 27: D_P -> unconnected-(U1-Pad27)
- U1 pad 28: COL13 -> unconnected-(U1-Pad28)
- U1 pad 29: COL14 -> unconnected-(U1-Pad29)
- U1 pad 3: ROTB -> unconnected-(U1-Pad3)
- U1 pad 30: COL15 -> unconnected-(U1-Pad30)
- U1 pad 37: unconnected-(U1-Pad37) -> COL4
- U1 pad 38: unconnected-(U1-Pad38) -> COL5
- U1 pad 39: unconnected-(U1-Pad39) -> COL6
- U1 pad 4: ROTA -> unconnected-(U1-Pad4)
- U1 pad 40: unconnected-(U1-Pad40) -> COL7
- U1 pad 41: COL4 -> ROW0
- U1 pad 42: LED_PWM -> unconnected-(U1-Pad42)
- U1 pad 43: COL5 -> unconnected-(U1-Pad43)
- U1 pad 44: unconnected-(U1-Pad44) -> D_N
- U1 pad 45: unconnected-(U1-Pad45) -> D_P
- U1 pad 46: COL6 -> unconnected-(U1-Pad46)
- U1 pad 49: COL7 -> unconnected-(U1-Pad49)
- U1 pad 5: COL10 -> ROW1
- U1 pad 50: ROW0 -> unconnected-(U1-Pad50)
- U1 pad 54: COL9 -> unconnected-(U1-Pad54)
- U1 pad 55: UGLED -> unconnected-(U1-Pad55)
- U1 pad 56: ROW1 -> unconnected-(U1-Pad56)
- U1 pad 57: ROW2 -> unconnected-(U1-Pad57)
- U1 pad 58: ROW3 -> unconnected-(U1-Pad58)
- U1 pad 59: ROW4 -> unconnected-(U1-Pad59)
- U1 pad 6: COL11 -> ROW2
- U1 pad 61: ROW5 -> unconnected-(U1-Pad61)
- U1 pad 62: COL8 -> unconnected-(U1-Pad62)
- U1 pad 8: COL16 -> ROW3
- U1 pad 9: COL17 -> ROW4
- U2 pad 2: +3V3 -> +3.3V
Routing:
- net +5V: track 0.00 -> 2202.1 mm, vias 0 -> 100
- net ROW0: track 0.00 -> 676.6 mm, vias 0 -> 22
- net ROW1: track 0.00 -> 531.3 mm, vias 0 -> 19
- net ROW2: track 0.00 -> 528.8 mm, vias 0 -> 19
- net ROW3: track 0.00 -> 455.4 mm, vias 0 -> 19
- net ROW4: track 0.00 -> 423.6 mm, vias 0 -> 19
- net ROW5: track 0.00 -> 388.9 mm, vias 0 -> 15
- net COL1: track 0.00 -> 327.4 mm, vias 0 -> 3
- net COL0: track 0.00 -> 313.3 mm, vias 0 -> 2
- net COL2: track 0.00 -> 305.9 mm, vias 0 -> 2
- net D_N: track 0.00 -> 303.5 mm
- net D_P: track 0.00 -> 302.4 mm
- net COL3: track 0.00 -> 287.1 mm, vias 0 -> 2
- net COL4: track 0.00 -> 262.1 mm, vias 0 -> 2
- net COL5: track 0.00 -> 241.0 mm, vias 0 -> 2
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Other:
- outline, holes or cut-outs redrawn

Commit message: Fix decoupling capacitor schematic for Voltage regulator + Some more routing
Parts:
- removed C12, C13, C14, C9: 100nF, Capacitor_SMD:C_0402_1005Metric
- removed C15, C16, C7: 4.7uF, Capacitor_SMD:C_0402_1005Metric
- removed C3, C4: 100uF, Capacitor_Tantalum_SMD:CP_EIA-3528-21_Kemet-B
- removed C6: 1uF, Capacitor_SMD:C_0402_1005Metric
- removed U2: XC6206P332MR, Package_TO_SOT_SMD:SOT-23
- added U3: XC6206P332MR, Package_TO_SOT_SMD:SOT-23, B.Cu at (-561.9, 129.5)
- C1, C17, R10, R100, R12, R16, R22, R24, R27, R28, R29, R34, R35, R38, R39, R41, R43, R46, R48, R49, R50, R51, R6, R61, R66, R68, R70, R71, R72, R76, R83, R86, R87, R9, R90, R92, R96: moved to B.Cu
- C5: value 10uF -> 1uF; footprint Capacitor_Tantalum_SMD:CP_EIA-3216-18_Kemet-A -> Capacitor_SMD:C_0402_1005Metric
- moved R10 687.0 mm to (-756.6, 100.3), turned to 180 degrees
- moved R12 665.4 mm to (-756.8, 138.5), turned to 180 degrees
- moved R9 663.0 mm to (-756.6, 81.3), turned to 180 degrees
- moved R28 652.5 mm to (-675.6, 100.3), turned to 180 degrees
- moved R16 649.1 mm to (-737.5, 119.4), turned to 180 degrees
- moved R34 633.9 mm to (-656.5, 100.4), turned to 180 degrees
- moved R22 628.4 mm to (-702.2, 100.3), turned to 180 degrees
- moved R24 623.4 mm to (-689.8, 28.9), turned to 180 degrees
- moved R29 587.1 mm to (-670.8, 28.9), turned to 180 degrees
- moved R41 584.7 mm to (-632.8, 62.2), turned to 180 degrees
- moved R27 582.8 mm to (-680.4, 81.3), turned to 180 degrees
- moved R43 580.5 mm to (-623.3, 81.3), turned to 180 degrees
- moved R38 571.8 mm to (-642.3, 81.3), turned to 180 degrees
- moved R15 571.7 mm to (-737.5, 100.3)
- moved C1 563.5 mm to (-601.6, 135.4), turned to 90 degrees
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Connections:
- U1 pad 57: unconnected-(U1-Pad57) -> COL8
- U1 pad 58: unconnected-(U1-Pad58) -> COL9
- U1 pad 59: unconnected-(U1-Pad59) -> COL10
Routing:
- net LED-: track 0.00 -> 2092.8 mm, vias 0 -> 103
- net +3.3V: track 20.2 -> 401.5 mm, vias 0 -> 8
- net +5V: track 2202.1 -> 2338.8 mm, vias 100 -> 102
- net COL8: track 120.4 -> 176.4 mm
- net /BOOT: track 9.37 -> 64.3 mm, vias 0 -> 2
- net COL10: track 100.4 -> 155.3 mm, vias 0 -> 2
- net COL9: track 100.4 -> 143.8 mm
- net GND: track 0.59 -> 24.4 mm, vias 0 -> 3
- net COL11: track 100.4 -> 105.8 mm
- net COL7: track 236.2 -> 241.3 mm
- net COL5: track 241.0 -> 245.0 mm
- net COL4: track 262.1 -> 265.8 mm
- net COL6: track 225.1 -> 228.3 mm
- net ROTA: track 0.00 -> 3.04 mm
- net ROTB: track 0.00 -> 3.01 mm
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